Commit message: Update robot.urdf

File: project3_description/urdf/robot.urdf (robot description, URDF)
Before this commit: robot my_robot, 6 links, 5 joints
Links:
- link base_link: geometry collision mesh filename=file:$(find project3_description)/models/Robot_Base_Chasis.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 scale=0.01 0.01 0.01; visual mesh filename=file:$(find project3_description)/models/Robot_Base_Chasis.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 scale=0.01 0.01 0.01
- link wheel1_link: geometry collision mesh filename=file:$(find project3_description)/models/Robot_Wheel.dae scale=0.01 0.01 0.01; visual mesh filename=file:$(find project3_description)/models/Robot_Wheel.dae scale=0.01 0.01 0.01
- link wheel2_link: geometry collision mesh filename=file:$(find project3_description)/models/Robot_Wheel.dae scale=0.01 0.01 0.01; visual mesh filename=file:$(find project3_description)/models/Robot_Wheel.dae scale=0.01 0.01 0.01
- link wheel3_link: geometry collision mesh filename=file:$(find project3_description)/models/Robot_Wheel.dae scale=0.01 0.01 0.01; visual mesh filename=file:$(find project3_description)models/Robot_Wheel.dae scale=0.01 0.01 0.01
- link wheel4_link: geometry collision mesh filename=file:$(find project3_description)/models/Robot_Wheel.dae scale=0.01 0.01 0.01; visual mesh filename=file:$(find project3_description)/models/Robot_Wheel.dae scale=0.01 0.01 0.01
